Commit message: Fix gripper URDF mesh paths for Isaac importer
Isaac's URDF importer ignores the MuJoCo meshdir hint and resolves mesh
filenames relative to the URDF, so bare base.stl/tip.stl failed to
resolve. Point them at meshes/ (and set mujoco meshdir="." for parity).

Conversion verified locally (RTX 3060, leisaac env): produces
linear_gripper.usd with bodies robotiq_base_link / left_inner_finger /
right_inner_finger and joints finger_joint / right_finger_joint, all
matching the 2F-85 contract. The URDF <mimic> did NOT survive import
(right_finger_joint is a free prismatic) -- will be coupled via
dual-drive (actuator + binary action drive both jaws), the idiomatic
Isaac Lab parallel-gripper approach, not a PhysX mimic.

File: source/uwlab_assets/uwlab_assets/local/Robots/LinearGripper/gripper.urdf (robot description, URDF)
Before this commit: robot linear_gripper, 3 links, 2 joints
Links:
- link left_inner_finger: geometry collision mesh filename=meshes/tip.stl scale=0.001 0.001 0.001; visual mesh filename=meshes/tip.stl scale=0.001 0.001 0.001
- link right_inner_finger: geometry collision mesh filename=meshes/tip.stl scale=0.001 0.001 0.001; visual mesh filename=meshes/tip.stl scale=0.001 0.001 0.001
- link robotiq_base_link: geometry collision mesh filename=meshes/base.stl scale=0.001 0.001 0.001; visual mesh filename=meshes/base.stl scale=0.001 0.001 0.001
