Commit message: Gripper base visual: include the camera-mount bracket + D405 (visual-only)
The RGB cameras must see the real gripper: base_visual.stl adds the printed
bracket and the D405 body to the base link's VISUAL mesh (2026-07-13).
Collision stays the original base.stl -- a new collider shape would grow the
per-shape material observation and break checkpoints trained before it, and
the bracket never touches the workspace in this top-down task.

File: source/uwlab_assets/uwlab_assets/local/Robots/LinearGripper/gripper.urdf (robot description, URDF)
Before this commit: robot linear_gripper, 3 links, 2 joints
Links:
- link robotiq_base_link: geometry collision mesh filename=meshes/base.stl scale=0.001 0.001 0.001; visual mesh filename=meshes/base_visual.stl scale=0.001 0.001 0.001
